File: Infra-pHAT.sch (KiCad schematic (older format))
At the start: 20 parts, among them Q1 BC817, U1 CAT24C32WI-GT3

Commit message: Initial version SCH + PCM
Parts:
- removed UART1: CONN_01X04, Pin_Headers:Pin_Header_Straight_1x04, symbol CONN_01X04
- added D1: 1N4148, Diodes_SMD:D_SOD-123, symbol D
- added J1: CONN_01X03, myfootprint:KLEMA_1x3, symbol CONN_01X03
- added P1: RAS-05-15, myfootprint:RAS-05-15, symbol RAS-05-15
- added Q2: BC817-40, TO_SOT_Packages_SMD:SOT-23, symbol BC817-40
- added R8: 2.7k, Resistors_SMD:R_0603_HandSoldering, symbol R
- added R9: 27k, Resistors_SMD:R_0603_HandSoldering, symbol R
- IRTX1, IRTX2: footprint LEDs:LED-5MM -> LEDs:LED_D5.0mm; symbol LED -> LED-RESCUE-Infra-pHAT
- JP1: footprint Pin_Headers:Pin_Header_Straight_1x02 -> Pin_Headers:Pin_Header_Straight_1x02_Pitch1.00mm
- RASP_CONN1: footprint Pin_Headers:Pin_Header_Straight_2x20 -> myfootprint:Pin_Header_Straight_2x20
- SENS1, SENS2, SENS3: footprint Pin_Headers:Pin_Header_Straight_1x04 -> Pin_Headers:Pin_Header_Straight_1x04_Pitch1.00mm
Connections:
- wire segments 56 -> 70
Other:
- moved on the sheet: C2, IRRX1, Q1, R4, R5
